Commit message: Wheely_Boi.xacro had unused transmission element

File: urdf/wheely_boi.xacro (robot description, xacro)
@@ -96,20 +96,4 @@
     <dynamics friction="0.1"/>
   </joint>
-  <transmission name="motorL">
-    <type>transmission_interfaxe/SimpleTransmission</type>
-    <actuator name="$l_motor">
-      <mechanicalReduction>1</mechanicalReduction>
-    </actuator>
-    <joint name="jointL">
-    </joint>
-  </transmission>
-  <transmission name="motorR">
-    <type>transmission_interfaxe/SimpleTransmission</type>
-    <actuator name="$r_motor">
-      <mechanicalReduction>1</mechanicalReduction>
-    </actuator>
-    <joint name="jointR">
-    </joint>
-  </transmission>
   <gazebo>
     <plugin name="wb_plugin" filename="libwb_plugin.so"> </plugin>

Commit message: Updated wheely_boi.xacro to remove all unneeded commands

File: urdf/wheely_boi.xacro (robot description, xacro)
@@ -7,14 +7,5 @@
   <xacro:property name="body_width" value="0.050" />
   <xacro:property name="body_length" value="0.035" />
-  <material name="blue">
-    <color rgba="0 0 0.8 1"/>
-  </material>
-  <material name="red">
-    <color rgba="0.8 0 0 1"/>
-  </material>
-  <material name="white">
-    <color rgba="1 1 1 1"/>
-  </material>
-  <gazebo reference="base_link">
+  <gazebo reference="edumip_body">
     <material>Gazebo/White</material>
     <mu1>0.2</mu1>
@@ -36,5 +27,4 @@
         <box size="${body_length} ${body_width} ${body_height}"/>
       </geometry>
-      <material name="white"/>
     </visual>
     <collision>
@@ -53,5 +43,4 @@
         <cylinder length="${wheel_width}" radius="${wheel_radius}"/>
       </geometry>
-      <material name="blue"/>
     </visual>
     <collision>
@@ -70,5 +59,4 @@
         <cylinder length="${wheel_width}" radius="${wheel_radius}"/>
       </geometry>
-      <material name="red"/>
     </visual>
     <collision>
