Commit message: Plugin at state of end of Lesson 3

File: urdf/rover.xacro (robot description, xacro)
@@ -23,5 +23,5 @@
     </collision>
     <inertial>
-      <mass value="5"/>
+      <mass value="15"/>
       <inertia ixx="${(5/12) * (body_width * body_width + body_height* body_height)}" ixy="0" ixz="0" iyy="${(5/12) * (body_length * body_length + body_height * body_height)}" iyz="0" izz="${(5/12) * (body_width * body_width + body_length * body_length)}" />
     </inertial>
@@ -50,5 +50,5 @@
     </link>
   </xacro:macro>
-  <xacro:wheel_link name="wFL" radius="${wheel_radius}" width="${wheel_width}" mass="0.3"/>
+  <xacro:wheel_link name="wFL" radius="${wheel_radius}" width="${wheel_width}" mass="2"/>
   <joint name="jFL" type="continuous">
     <parent link="body"/>
@@ -56,7 +56,7 @@
     <axis xyz="0 0 1"/>
     <origin xyz="${body_length/2 - 0.03} ${body_width/2 + wheel_width/2} 0" rpy="${pi/2} 0 0" />
-    <dynamics friction="0.1"/>
+    <dynamics friction="0.5"/>
   </joint>
-  <xacro:wheel_link name="wBL" radius="${wheel_radius}" width="${wheel_width}" mass="0.3"/>
+  <xacro:wheel_link name="wBL" radius="${wheel_radius}" width="${wheel_width}" mass="2"/>
   <joint name="jBL" type="continuous">
     <parent link="body"/>
@@ -64,7 +64,7 @@
     <axis xyz="0 0 1"/>
     <origin xyz="-${body_length/2 - 0.03} ${body_width/2 + wheel_width/2} 0" rpy="${pi/2} 0 0" />
-    <dynamics friction="0.1"/>
+    <dynamics friction="0.5"/>
   </joint>
-  <xacro:wheel_link name="wFR" radius="${wheel_radius}" width="${wheel_width}" mass="0.3"/>
+  <xacro:wheel_link name="wFR" radius="${wheel_radius}" width="${wheel_width}" mass="2"/>
   <joint name="jFR" type="continuous">
     <parent link="body"/>
@@ -72,7 +72,7 @@
     <axis xyz="0 0 1"/>
     <origin xyz="${body_length/2 - 0.03} -${body_width/2 + wheel_width/2} 0" rpy="${pi/2} 0 0" />
-    <dynamics friction="0.1"/>
+    <dynamics friction="0.5"/>
   </joint>
-  <xacro:wheel_link name="wBR" radius="${wheel_radius}" width="${wheel_width}" mass="0.3"/>
+  <xacro:wheel_link name="wBR" radius="${wheel_radius}" width="${wheel_width}" mass="2"/>
   <joint name="jBR" type="continuous">
     <parent link="body"/>
@@ -80,5 +80,5 @@
     <axis xyz="0 0 1"/>
     <origin xyz="-${body_length/2 - 0.03} -${body_width/2 + wheel_width/2} 0" rpy="${pi/2} 0 0" />
-    <dynamics friction="0.1"/>
+    <dynamics friction="0.5"/>
   </joint>
   <gazebo>

Commit message: Differentials and controls beginning to be implemented

File: urdf/rover.xacro (robot description, xacro)
@@ -6,9 +6,12 @@
   <xacro:property name="body_width" value="0.15" />
   <xacro:property name="body_length" value="0.4" />
+  <xacro:property name="leg_height" value="0.05" />
+  <xacro:property name="leg_width" value="0.02" />
+  <xacro:property name="leg_length" value="0.02" />
   <gazebo reference="body">
     <material>Gazebo/White</material>
     <mu1>0.2</mu1>
     <mu2>0.2</mu2>
-  </gazebo>
+ </gazebo>
   <link name="body">
     <visual>
@@ -23,8 +26,52 @@
     </collision>
     <inertial>
-      <mass value="15"/>
+      <mass value="5"/>
       <inertia ixx="${(5/12) * (body_width * body_width + body_height* body_height)}" ixy="0" ixz="0" iyy="${(5/12) * (body_length * body_length + body_height * body_height)}" iyz="0" izz="${(5/12) * (body_width * body_width + body_length * body_length)}" />
     </inertial>
   </link>
+  <link name="lLeg">
+    <visual>
+      <geometry>
+        <box size="${leg_length} ${leg_width} ${leg_height}"/>
+      </geometry>
+    </visual>
+    <collision>
+      <geometry>
+        <box size="${leg_length} ${leg_width} ${leg_height}"/>
+      </geometry>
+    </collision>
+    <inertial>
+      <mass value="1"/>
+      <inertia ixx="${(1/12) * (leg_width * leg_width + leg_height* leg_height)}" ixy="0" ixz="0" iyy="${(1/12) * (leg_length * leg_length + leg_height * leg_height)}" iyz="0" izz="${(1/12) * (leg_width * leg_width + leg_length * leg_length)}" />
+    </inertial>
+  </link>
+  <joint name="lDifJoint" type="continuous">
+    <parent link="body"/>
+    <child link="lLeg"/>
+    <axis xyz="0 0 1"/>
+    <origin xyz="${body_length/2 - 0.03} ${body_width/2 + wheel_width/2} -${body_height/2}"/>
+  </joint>
+  <link name="rLeg">
+    <visual>
+      <geometry>
+        <box size="${leg_length} ${leg_width} ${leg_height}"/>
+      </geometry>
+    </visual>
+    <collision>
+      <geometry>
+        <box size="${leg_length} ${leg_width} ${leg_height}"/>
+      </geometry>
+    </collision>
+    <inertial>
+      <mass value="1"/>
+      <inertia ixx="${(1/12) * (leg_width * leg_width + leg_height* leg_height)}" ixy="0" ixz="0" iyy="${(1/12) * (leg_length * leg_length + leg_height * leg_height)}" iyz="0" izz="${(1/12) * (leg_width * leg_width + leg_length * leg_length)}" />
+    </inertial>
+  </link>
+  <joint name="rDifJoint" type="continuous">
+    <parent link="body"/>
+    <child link="rLeg"/>
+    <axis xyz="0 0 1"/>
+    <origin xyz="${body_length/2 - 0.03} -${body_width/2 + wheel_width/2} -${body_height/2}"/>
+  </joint>
   <xacro:macro name="wheel_link" params="name radius width mass">
     <gazebo reference="${name}">
@@ -32,5 +79,5 @@
       <mu1>0.84</mu1>
       <mu2>0.84</mu2>
-    </gazebo>
+   </gazebo>
     <link name="${name}">
       <visual>
@@ -52,8 +99,8 @@
   <xacro:wheel_link name="wFL" radius="${wheel_radius}" width="${wheel_width}" mass="2"/>
   <joint name="jFL" type="continuous">
-    <parent link="body"/>
+    <parent link="lLeg"/>
     <child link="wFL"/>
     <axis xyz="0 0 1"/>
-    <origin xyz="${body_length/2 - 0.03} ${body_width/2 + wheel_width/2} 0" rpy="${pi/2} 0 0" />
+    <origin xyz="0 ${leg_width/2} ${leg_length/2}" rpy="${pi/2} 0 0" />
     <dynamics friction="0.5"/>
   </joint>
@@ -68,8 +115,8 @@
   <xacro:wheel_link name="wFR" radius="${wheel_radius}" width="${wheel_width}" mass="2"/>
   <joint name="jFR" type="continuous">
-    <parent link="body"/>
+    <parent link="rLeg"/>
     <child link="wFR"/>
     <axis xyz="0 0 1"/>
-    <origin xyz="${body_length/2 - 0.03} -${body_width/2 + wheel_width/2} 0" rpy="${pi/2} 0 0" />
+    <origin xyz="0 -${leg_width/2} ${leg_length/2}" rpy="${pi/2} 0 0" />
     <dynamics friction="0.5"/>
   </joint>
